File: feather-mikrobus.kicad_pcb (KiCad board)
At the start: 2 copper layers, 63.5 x 58.4 mm, 24 parts, among them J1 FEATHER-HEADER-16POS-PTH, J2 FEATHER-HEADER-12POS-PTH, J3 MIKROBUS-HEADER-LEFT-PTH, J4 MIKROBUS-HEADER-RIGHT-PTH, SW1 JS102011SAQN, SW2 KMR421GULCLFS, SW3 KMR421GULCLFS

Commit message: Change names
Parts:
- A1: value FEATHER-MODULE -> Adafruit_Feather_socket_empty; footprint Flying_Camp_Design:FEATHER-MODULE -> Flying_Camp_Design:Adafruit_Feather_socket_empty
- A2: value MIKROBUS-MODULE -> mikroBUS_socket_empty; footprint Flying_Camp_Design:MIKROBUS-MODULE -> Flying_Camp_Design:mikroBUS_socket_empty
- FID1, FID2, FID3: value FIDUCIAL -> Fiducial_1mm_Mask2mm
- J1: value FEATHER-HEADER-16POS-PTH -> Adafruit_Feather_socket_header_left_pth; footprint Flying_Camp_Design:FEATHER-HEADER-16POS-PTH -> Flying_Camp_Design:Adafruit_Feather_socket_header_left_pth
- J2: value FEATHER-HEADER-12POS-PTH -> Adafruit_Feather_socket_header_right_pth; footprint Flying_Camp_Design:FEATHER-HEADER-12POS-PTH -> Flying_Camp_Design:Adafruit_Feather_socket_header_right_pth
- J3: value MIKROBUS-HEADER-LEFT-PTH -> mikroBUS_socket_header_left_pth; footprint Flying_Camp_Design:MIKROBUS-HEADER-LEFT-PTH -> Flying_Camp_Design:mikroBUS_socket_header_left_pth
- J4: value MIKROBUS-HEADER-RIGHT-PTH -> mikroBUS_socket_header_right_pth; footprint Flying_Camp_Design:MIKROBUS-HEADER-RIGHT-PTH -> Flying_Camp_Design:mikroBUS_socket_header_right_pth
- LOGO1: value MIKROBUS_LOGO -> mikroBUS_logo
- LOGO3: value FEATHER-LOGO -> Adafruit_Feather_logo; footprint Flying_Camp_Design:FEATHER-LOGO -> Flying_Camp_Design:Adafruit_Feather_logo
- MH1: value FEATHER-MOUNTING-HOLES -> Adafruit_Feather_socket_mounting_holes; footprint Flying_Camp_Design:FEATHER-MOUNTING-HOLES -> Flying_Camp_Design:Adafruit_Feather_socket_mounting_holes
Changed lines of the file:
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@@
     )
   )
-  (module Flying_Camp_Design:FEATHER-MODULE (layer F.Cu)
+  (module Flying_Camp_Design:Adafruit_Feather_socket_empty (layer F.Cu)
     (at 171.45 100.33)
     (descr "Adafruit Feather plug-in module")
@@
       (effects (font (size 1 1) (thickness 0.15)))
     )
-    (fp_text value FEATHER-MODULE (at 0 0 unlocked) (layer F.Fab) hide
+    (fp_text value Adafruit_Feather_socket_empty (at 0 0 unlocked) (layer F.Fab) hide
       (effects (font (size 1 1) (thickness 0.15)))
     )
@@
     (pad 5 smd rect (at 0 -1.425 270) (size 1.7 0.55) (layers F.Cu F.Paste F.Mask)
       (net 1 GND))
-    (model :Flying_Camp_Design:KMR421GULCLFS.STEP
+    (model :Flying_Camp_Design:KMR421GULCLFS.step
       (offset (xyz 0 0 1.4))
       (scale (xyz 1 1 1))
@@
     )
   )
-  (module Flying_Camp_Design:MIKROBUS-MODULE (layer F.Cu)
+  (module Flying_Camp_Design:mikroBUS_socket_empty (layer F.Cu)
     (at 186.69 128.27 90)
     (fp_text reference A2 (at 0 0 90 unlocked) (layer F.SilkS)
       (effects (font (size 1 1) (thickness 0.15)))
     )
-    (fp_text value MIKROBUS-MODULE (at 0 0 90 unlocked) (layer F.Fab) hide
+    (fp_text value mikroBUS_socket_empty (at 0 0 90 unlocked) (layer F.Fab) hide
       (effects (font (size 1 1) (thickness 0.15)))
     )
@@
     (pad 5 smd rect (at 0 -1.425 270) (size 1.7 0.55) (layers F.Cu F.Paste F.Mask)
       (net 1 GND))
-    (model :Flying_Camp_Design:KMR421GULCLFS.STEP
+    (model :Flying_Camp_Design:KMR421GULCLFS.step
       (offset (xyz 0 0 1.4))
       (scale (xyz 1 1 1))
@@
     )
   )
-  (module Flying_Camp_Design:FEATHER-LOGO (layer F.Cu)
+  (module Flying_Camp_Design:Adafruit_Feather_logo (layer F.Cu)
     (at 156.21 97.155 90)
     (attr virtual)
@@
       (effects (font (size 1.524 1.524) (thickness 0.3)))
     )
-    (fp_text value FEATHER-LOGO (at 0.75 0 90) (layer F.SilkS) hide
+    (fp_text value Adafruit_Feather_logo (at 0.75 0 90) (layer F.SilkS) hide
       (effects (font (size 1.524 1.524) (thickness 0.3)))
     )
@@
       (effects (font (size 1 1) (thickness 0.15)))
     )
-    (fp_text value FIDUCIAL (at 0 2) (layer F.Fab) hide
+    (fp_text value Fiducial_1mm_Mask2mm (at 0 2) (layer F.Fab) hide
       (effects (font (size 1 1) (thickness 0.15)))
     )
@@
       (effects (font (size 1 1) (thickness 0.15)))
     )
-    (fp_text value FIDUCIAL (at 0 2) (layer F.Fab) hide
+    (fp_text value Fiducial_1mm_Mask2mm (at 0 2) (layer F.Fab) hide
       (effects (font (size 1 1) (thickness 0.15)))
     )
@@
       (effects (font (size 1 1) (thickness 0.15)))
     )
-    (fp_text value FIDUCIAL (at 0 2) (layer F.Fab) hide
+    (fp_text value Fiducial_1mm_Mask2mm (at 0 2) (layer F.Fab) hide
       (effects (font (size 1 1) (thickness 0.15)))
     )
@@
       (effects (font (size 1 1) (thickness 0.15)))
     )
-    (fp_text value MIKROBUS_LOGO (at 0.75 -12.7 90) (layer F.Fab) hide
+    (fp_text value mikroBUS_logo (at 0.75 -12.7 90) (layer F.Fab) hide
       (effects (font (size 1 1) (thickness 0.15)))
     )
@@
     )
   )
-  (module Flying_Camp_Design:FEATHER-HEADER-16POS-PTH (layer F.Cu)
+  (module Flying_Camp_Design:Adafruit_Feather_socket_header_left_pth (layer F.Cu)
     (at 171.45 100.33 90)
     (descr "Through hole straight socket strip, 1x16, 2.54mm pitch, single row (from Kicad 4.0.7), script generated")
@@
       (effects (font (size 1 1) (thickness 0.15)))
     )
-    (fp_text value FEATHER-HEADER-16POS-PTH (at -10.16 21.82 90 unlocked) (layer F.Fab) hide
+    (fp_text value Adafruit_Feather_socket_header_left_pth (at -10.16 21.82 90 unlocked) (layer F.Fab) hide
       (effects (font (size 1 1) (thickness 0.15)))
     )
@@
       (net 2 +3V3))
     (pad ~RST thru_hole rect (at -10.16 -19.05 90) (size 1.7 1.7) (drill 1) (layers *.Cu *.Mask))
-    (model :Flying_Camp_Design:FEATHER-HEADER-16POS-PTH.wrl
+    (model :Flying_Camp_Design:Adafruit_Feather_socket_header_left_pth.wrl
       (offset (xyz -10.16 19.05 0))
       (scale (xyz 1 1 1))
@@
     )
   )
-  (module Flying_Camp_Design:FEATHER-HEADER-12POS-PTH (layer F.Cu)
+  (module Flying_Camp_Design:Adafruit_Feather_socket_header_right_pth (layer F.Cu)
     (at 171.45 100.33 90)
     (descr "Through hole straight socket strip, 1x12, 2.54mm pitch, single row (from Kicad 4.0.7), script generated")
@@
       (effects (font (size 1 1) (thickness 0.15)))
     )
-    (fp_text value FEATHER-HEADER-12POS-PTH (at 10.16 21.82 90 unlocked) (layer F.Fab) hide
+    (fp_text value Adafruit_Feather_socket_header_right_pth (at 10.16 21.82 90 unlocked) (layer F.Fab) hide
       (effects (font (size 1 1) (thickness 0.15)))
     )
@@
       (net 11 /FEATHER_EN))
     (pad VBAT thru_hole rect (at 10.16 -8.89 90) (size 1.7 1.7) (drill 1) (layers *.Cu *.Mask))
-    (model :Flying_Camp_Design:FEATHER-HEADER-12POS-PTH.wrl
+    (model :Flying_Camp_Design:Adafruit_Feather_socket_header_right_pth.wrl
       (offset (xyz 10.16 8.890000000000001 0))
       (scale (xyz 1 1 1))
@@
       (net 11 /FEATHER_EN))
     (pad 1 smd rect (at -2.5 -2.75 270) (size 1.25 2.5) (layers F.Cu F.Paste F.Mask))
-    (model :Flying_Camp_Design:JS102011SAQN.STEP
+    (model :Flying_Camp_Design:JS102011SAQN.step
       (offset (xyz 0 0 0.2794))
       (scale (xyz 1 1 1))
@@
     )
   )
-  (module Flying_Camp_Design:MIKROBUS-HEADER-RIGHT-PTH (layer F.Cu)
+  (module Flying_Camp_Design:mikroBUS_socket_header_right_pth (layer F.Cu)
     (at 186.69 128.27 90)
     (descr "Through hole straight pin header, 1x08, 2.54mm pitch, single row")
@@
       (effects (font (size 1 1) (thickness 0.15)))
     )
-    (fp_text value MIKROBUS-HEADER-RIGHT-PTH (at 0 0 90 unlocked) (layer F.Fab) hide
+    (fp_text value mikroBUS_socket_header_right_pth (at 0 0 90 unlocked) (layer F.Fab) hide
       (effects (font (size 1 1) (thickness 0.15)))
     )
@@
     )
   )
-  (module Flying_Camp_Design:MIKROBUS-HEADER-LEFT-PTH (layer F.Cu)
+  (module Flying_Camp_Design:mikroBUS_socket_header_left_pth (layer F.Cu)
     (at 186.69 128.27 90)
     (descr "Through hole straight pin header, 1x08, 2.54mm pitch, single row")
@@
       (effects (font (size 1 1) (thickness 0.15)))
     )
-    (fp_text value MIKROBUS-HEADER-LEFT-PTH (at 0 0 90 unlocked) (layer F.Fab) hide
+    (fp_text value mikroBUS_socket_header_left_pth (at 0 0 90 unlocked) (layer F.Fab) hide
       (effects (font (size 1 1) (thickness 0.15)))
     )
@@
     )
   )
-  (module Flying_Camp_Design:FEATHER-MOUNTING-HOLES (layer F.Cu)
+  (module Flying_Camp_Design:Adafruit_Feather_socket_mounting_holes (layer F.Cu)
     (at 171.45 100.33)
     (descr "Mounting holes for Adafruit Feather")
@@
       (effects (font (size 1 1) (thickness 0.15)))
     )
-    (fp_text value FEATHER-MOUNTING-HOLES (at 0 0) (layer F.Fab) hide
-      (effects (font (size 1 1) (thickness 0.15)))
-    )
+    (fp_text value Adafruit_Feather_socket_mounting_holes (at 0 0) (layer F.Fab) hide
+      (effects (font (size 1 1) (thickness 0.15)))
+    )

Commit message: Finish schematic and board routing for V1
Parts:
- added D2: LTST-C191KGKT, Flying_Camp_Design:LED_0603_1608Metric, F.Cu at (142.9, 118.1)
- added R8: RC0603JR-07330RL, Flying_Camp_Design:R_0603_1608Metric, F.Cu at (142.9, 120.0)
- added REF**: OSHW-Logo2_14.6x12mm_SilkScreen, Flying_Camp_Design:OSHW-Logo2_14.6x12mm_SilkScreen, F.Cu at (157.5, 124.5)
- added REF**: KiCad-Logo_5mm_SilkScreen, Flying_Camp_Design:KiCad-Logo_5mm_SilkScreen, F.Cu at (157.5, 134.6)
- J1: value Adafruit_Feather_socket_header_left_pth -> PinSocket_1x16_P2.54mm_Vertical
- J2: value Adafruit_Feather_socket_header_right_pth -> PinSocket_1x12_P2.54mm_Vertical
- moved R2 8.25 mm to (142.9, 125.1)
- moved D1 4.44 mm to (142.9, 123.2)
- moved R7 1.08 mm to (148.7, 103.6), turned to 270 degrees
- moved LOGO3 0.64 mm to (155.6, 97.2)
Routing:
- net GND: track 21.4 -> 32.1 mm
- net /~USER_LED: track 48.0 -> 50.7 mm
- net Net-(D2-Pad2): track 0.00 -> 1.91 mm
- net Net-(R7-Pad1): track 2.64 -> 4.18 mm
- net /FEATHER_EN: track 26.1 -> 24.7 mm
- net /MIKROBUS_PWM: track 31.3 -> 30.1 mm
- net /MOSI: track 37.8 -> 37.1 mm
- net /USER_SW: track 51.1 -> 50.4 mm
- net Net-(D1-Pad2): track 2.54 -> 1.91 mm
Other:
- board text added: "Feather mikroBUS V1"
- board text added: "FlyingCamp.Design"
