File: hardware/feather-mikrobus-v1/feather-mikrobus-v1.kicad_pcb (KiCad board)
At the start: 2 copper layers, 63.5 x 58.4 mm, 27 parts, among them J1 Adafruit_Feather_socket_heade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, J2 Adafruit_Feather_socket_heade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, J3 mikroBUS_socket_header_left_p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, J4 mikroBUS_socket_header_right_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, SW1 C_and_K_JS102011SAQN, SW2 C_and_K_KMR421GULCLFS, SW3 C_and_K_KMR421GULCLFS

Commit message: Upgrade design to KiCad 5.99
Other:
- net class Default removed
- net class Power removed

Commit message: Revert "Upgrade design to KiCad 5.99"
This reverts commit 404d8fe5192a3f2d218e68c3ca65a2b30fdaee8b.
Other:
- net class Default added: clearance 0.1524, trace_width 0.1524, via_dia 0.508, via_drill 0.254
- net class Power added: clearance 0.1524, trace_width 0.381, via_dia 0.508, via_drill 0.254
